File: hw/RTC-Clock-Display-Led-7Seg.kicad_pcb (KiCad board)
At the start: 2 copper layers, 210 x 70 mm, 89 parts, among them IC1 STM8S003F3P, J1 BARREL_JACK, J2 DS18B20, J4 CONN_01X04, Q1 A1015, Q10 C1815, Q2 A1015, Q3 A1015, Q4 A1015, Q5 C1815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

Commit message: upload
Parts:
- moved Q1 51.8 mm to (180.1, 101.1)
- moved Q5 51.8 mm to (170.6, 101.3)
- moved R16 51.8 mm to (176.9, 101.1)
- moved R21 51.8 mm to (167.1, 101.6)
- moved R9 51.8 mm to (174.1, 101.1)
- moved R14 34.9 mm to (233.5, 64.9)
- moved R36 34.5 mm to (241.5, 55.0)
- moved J2 34.3 mm to (245.5, 58.8)
- moved D5 33.4 mm to (229.0, 63.8), turned to 180 degrees
- moved C12 32.5 mm to (226.2, 80.0), turned to 90 degrees
- moved C11 28.2 mm to (227.9, 68.2), turned to 90 degrees
- moved C9 21.5 mm to (219.2, 81.1), turned to 180 degrees
- moved R2 19.5 mm to (223.4, 86.8)
- moved D2 18.6 mm to (218.4, 87.0)
- moved R6 18.3 mm to (226.2, 74.1), turned to 90 degrees
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Routing:
- net GND: track 0.00 -> 162.5 mm, vias 0 -> 2
- net +5V: track 0.00 -> 31.7 mm
- net +12V: track 0.00 -> 20.6 mm
- net Net-(D3-Pad1): track 0.00 -> 18.7 mm
- net Net-(R3-Pad1): track 0.00 -> 13.0 mm, vias 0 -> 2
- net /bt3: track 0.00 -> 11.9 mm
- net /bt1: track 0.00 -> 11.4 mm
- net /bt2: track 0.00 -> 10.8 mm
- net Net-(R1-Pad2): track 0.00 -> 10.1 mm
- net VIN: track 0.00 -> 7.93 mm
- net Net-(C8-Pad1): track 0.00 -> 5.86 mm
- net /ds18b20: track 0.00 -> 4.06 mm

Commit message: complete layout
Parts:
- moved C13 141.0 mm to (234.5, 84.5), turned to 90 degrees
- moved R22 136.2 mm to (191.9, 91.0), turned to 90 degrees
- moved C14 135.5 mm to (228.7, 84.5), turned to 90 degrees
- moved Y1 130.9 mm to (231.6, 83.7), turned to 0 degrees
- moved Q6 129.4 mm to (188.4, 91.0), turned to 270 degrees
- moved R11 122.8 mm to (185.2, 91.0), turned to 90 degrees
- moved C15 120.9 mm to (225.6, 77.9), turned to 320 degrees
- moved BT1 120.4 mm to (223.3, 73.9), turned to 50 degrees
- moved R17 118.1 mm to (183.0, 91.0), turned to 90 degrees
- moved C17 113.0 mm to (222.3, 81.1), turned to 0 degrees
- moved U4 112.7 mm to (222.2, 84.9), turned to 180 degrees
- moved Q2 111.6 mm to (179.6, 90.9), turned to 270 degrees
- moved R34 98.9 mm to (215.9, 78.6)
- moved R35 98.9 mm to (213.6, 78.6)
- moved R23 87.4 mm to (192.0, 96.2), turned to 90 degrees
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Connections:
- IC1 pad 10: /l3 -> /l1
- IC1 pad 19: /bt1 -> /bt3
- IC1 pad 20: /bt2 -> /bt1
- IC1 pad 3: /bt3 -> /bt2
- IC1 pad 5: /l1 -> /l3
- U1 pad 1: Net-(U1-Pad1) -> /QH
- U1 pad 11: /DP -> /A
- U1 pad 12: /G -> /B
- U1 pad 13: /F -> /C
- U1 pad 14: /E -> /D
- U1 pad 15: /D -> /E
- U1 pad 16: /C -> /F
- U1 pad 17: /B -> /G
- U1 pad 18: /A -> /DP
- U1 pad 2: Net-(U1-Pad2) -> /QG
- U1 pad 3: Net-(U1-Pad3) -> /QF
- U1 pad 4: Net-(U1-Pad4) -> /QE
- U1 pad 5: Net-(U1-Pad5) -> /QD
- U1 pad 6: Net-(U1-Pad6) -> /QC
- U1 pad 7: Net-(U1-Pad7) -> /QB
- U1 pad 8: Net-(U1-Pad8) -> /QA
- U3 pad 1: Net-(U1-Pad2) -> /QB
- U3 pad 15: Net-(U1-Pad1) -> /QA
- U3 pad 16: VCC -> +5V
- U3 pad 2: Net-(U1-Pad3) -> /QC
- U3 pad 3: Net-(U1-Pad4) -> /QD
- U3 pad 4: Net-(U1-Pad5) -> /QE
- U3 pad 5: Net-(U1-Pad6) -> /QF
- U3 pad 6: Net-(U1-Pad7) -> /QG
- U3 pad 7: Net-(U1-Pad8) -> /QH
- Y1 pad 1: Net-(C13-Pad2) -> Net-(C14-Pad2)
- Y1 pad 2: Net-(C14-Pad2) -> Net-(C13-Pad2)
Routing:
- net +5V: track 31.7 -> 314.5 mm, vias 0 -> 23
- net GND: track 162.5 -> 386.7 mm, vias 2 -> 12
- net Net-(7SEG1-Pad6): track 0.00 -> 196.2 mm, vias 0 -> 1
- net Net-(7SEG1-Pad2): track 172.1 -> 335.7 mm, vias 0 -> 6
- net Net-(7SEG1-Pad3): track 173.4 -> 325.4 mm, vias 0 -> 4
- net Net-(7SEG1-Pad4): track 170.7 -> 315.6 mm, vias 0 -> 6
- net /led1: track 0.00 -> 144.7 mm
- net +12V: track 20.6 -> 147.6 mm, vias 0 -> 8
- net /led2: track 0.00 -> 84.8 mm
- net Net-(R32-Pad1): track 0.00 -> 82.9 mm, vias 0 -> 3
- net /ds18b20: track 4.06 -> 78.9 mm, vias 0 -> 4
- net /dot: track 0.00 -> 70.5 mm
- net /led4: track 0.00 -> 64.8 mm
- net /bt3: track 11.9 -> 56.1 mm, vias 0 -> 2
- net /led3: track 0.00 -> 41.0 mm
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- added copper zone on B.Cu, net +5V
- added copper zone on F.Cu, net +5V
- added copper zone on F.Cu, net Net-(7SEG1-Pad2)
- added copper zone on B.Cu, net Net-(7SEG1-Pad4)

Commit message: complete hw
Parts:
- added REF**: Vit-4mm, nhantt-kicad-lib:Vit-4mm, F.Cu at (145.0, 55.0)
- added REF**: Vit-4mm, nhantt-kicad-lib:Vit-4mm, F.Cu at (145.0, 115.0)
Routing:
- net GND: track 386.7 -> 800.3 mm, vias 12 -> 109
- net Net-(R32-Pad1): track 82.9 -> 76.4 mm
- net Net-(7SEG1-Pad7): track 202.5 -> 206.7 mm, vias 1 -> 2
- net Net-(7SEG1-Pad9): track 196.2 -> 199.8 mm, vias 1 -> 2
- net Net-(7SEG1-Pad10): track 180.7 -> 184.1 mm, vias 5 -> 6
- net Net-(7SEG1-Pad6): track 196.2 -> 199.2 mm, vias 1 -> 2
- net Net-(7SEG1-Pad2): track 335.7 -> 338.0 mm
- net /ds18b20: track 78.9 -> 80.9 mm, vias 4 -> 5
- net Net-(7SEG1-Pad3): track 325.4 -> 327.4 mm
- net /l4: track 32.2 -> 33.8 mm, vias 2 -> 4
- net /l2: track 19.4 -> 20.8 mm, vias 2 -> 4
- net Net-(7SEG1-Pad4): track 315.6 -> 317.0 mm
- net Net-(R3-Pad1): track 13.0 -> 14.4 mm, vias 2 -> 5
- net +12V: track 147.6 -> 148.9 mm, vias 8 -> 14
- net /latch: track 36.8 -> 35.6 mm
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- added copper zone on B.Cu, net +12V
- added copper zone on B.Cu, net /l1
- added copper zone on B.Cu, net /l2
- added copper zone on B.Cu, net /l3
- added copper zone on B.Cu, net /l4
- added copper zone on B.Cu, net GND
- added copper zone on F.Cu, net GND
- added copper zone on B.Cu, net Net-(7SEG1-Pad10)
- added copper zone on B.Cu, net Net-(7SEG1-Pad6)
- added copper zone on B.Cu, net Net-(7SEG1-Pad7)
- added copper zone on B.Cu, net Net-(7SEG1-Pad9)
- added copper zone on B.Cu, net Net-(BT1-Pad1)
- added copper zone on B.Cu, net Net-(D3-Pad1)
- added copper zone on B.Cu, net Net-(R1-Pad2)
- added copper zone on B.Cu, net Net-(R3-Pad1)
- added copper zone on B.Cu, net VIN
